File: PCB_Sensor_Board_2.x_HX711_DS18b20/Sensor_Board_2.01_HX711_DS18b2.brd (EAGLE design)
At the start: 40 x 70 mm, 26 parts

Commit message: add_ 1x DS18B20 TO-92
Parts:
- added DS18B20: DS2405, maxim:TO92-
Connections:
- net 3V3: now also DS18B20.3
- net DS18B20_DATA_GPIO11_PIN23: now also DS18B20.2
- net GND: now also DS18B20.1
Routing:
- net DS18B20_DATA_GPIO11_PIN23: track 55.6 -> 89.9 mm
- net 3V3: track 53.6 -> 77.3 mm
- net GND: track 138.1 -> 151.0 mm
- net HX711_V: track 49.2 -> 53.7 mm, vias 0 -> 1
- net E+: track 77.2 -> 78.9 mm
- net B-: track 31.8 -> 33.5 mm
- net HX711-SCK: track 17.4 -> 18.3 mm
