File: PCB_Sensor_Board_2.x_HX711_DS18b20/Sensor_Board_2.03_HX711_DS18b2.brd (EAGLE design)
At the start: 40 x 70 mm, 29 parts

Commit message: cleaning: old files ->  \old\
Routing:
- net GND: track 0.00 -> 162.0 mm
- net DS18B20_DATA_GPIO11_PIN23: track 0.00 -> 81.6 mm
- net E-: track 0.00 -> 80.8 mm
- net E+: track 0.00 -> 79.0 mm
- net 3V3: track 0.00 -> 78.0 mm
- net B-: track 0.00 -> 35.0 mm
- net HX711_V: track 0.00 -> 34.6 mm
- net B+: track 0.00 -> 22.2 mm
- net HX711-DT: track 0.00 -> 18.2 mm
- net A+: track 0.00 -> 17.9 mm
- net A-: track 0.00 -> 17.9 mm
- net HX711-SCK: track 0.00 -> 17.4 mm
- net N$4: track 0.00 -> 6.65 mm
- net N$3: track 0.00 -> 3.81 mm
- net N$2: track 0.00 -> 2.87 mm
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