File: PCB_V2.x/HoneyPI_Platine 2.01.brd (EAGLE design)
At the start: 80 x 100 mm, 74 parts

Commit message: only small changes :-)
Parts:
- removed 0#76/77: (no value), pinhead:1X02
- removed 5V(ALTERN.), JP_3V3_GPIO9, JP_3V3_RPI/LM33_G3, LM33CV_G2, LM33CV_G3: (no value), pinhead:1X03
- removed C_SP4, C_SP5, C_SP6: 100µF, capacitor-wima:C2.5-3
- added #76_77: (no value), pinhead:1X02
- added 32, C1: 10µF, rcl:E2-5
- added 5V(ALTERN.IN), 5V(OUT), DS18_3V3/GPIO9, HX711_RPI/LM33: (no value), pinhead:1X03
- added C_HC711_1: 0,1µF, capacitor-wima:C2.5-3
- added HX: (no value), pinhead:1X01
- added LM33_HX711, LM33_I²C: (no value), LM33cv:337TS
- added U$10, U$11, U$12, U$7, U$9: (no value), holes:3,0
- C_I²C_1: value 100µF -> 0,1µF
- C_TASTER: value 470nF -> 100nF
- R_TASTER: value 50K -> 47K
- moved JP_VORW 10.8 mm to (59.7, 64.8)
- moved R2_PCF8591 9.25 mm to (57.1, 14.0), turned to 0 degrees
- moved R_LED 8.13 mm to (59.7, 61.0)
- moved R_DS18B20 8.13 mm to (14.0, 39.4), turned to 270 degrees
- moved C_SP1 7.62 mm to (11.4, 26.7), turned to 270 degrees
- moved C_SP2 7.62 mm to (19.1, 26.7), turned to 270 degrees
- moved R1_PCF8591 6.84 mm to (63.5, 17.8), turned to 0 degrees
- moved HX711-2 6.05 mm to (36.4, 82.5)
- moved HX711-3 5.39 mm to (50.8, 82.5)
- moved SEEED2 5.23 mm to (36.3, 77.5)
- moved C_TASTER 4.58 mm to (68.6, 57.1)
- moved R_TASTER 4.58 mm to (59.7, 57.1)
- moved SEEED3 4.58 mm to (50.8, 77.5)
- moved HX711-5 4.02 mm to (17.8, 69.8)
- moved SEEED5 3.86 mm to (17.9, 64.9)
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- renumbered C_SP3 to C_I²C_1, JP_3V3_RPI/LM33_G2 to I²C_RPI/LM33
Connections:
- removed net GND_2: 0#76/77.1, BME680.2, BME680_GROVE.4, C_I²C_1.2, C_SP4.2, C_SP5.2, C_SP6.2, C_TASTER.1, DS1.4, DS18B20(T0-92).1, DS18B20-1.3, DS18B20-2.3, DS18B20-3.3, DS18B20-4.3, DS18B20-5.3, DS18B20-6.3, DS18B20-7.3, DS18B20-8.3, DS2.4, DS3.4, DS4.4, DS5.4, DS6.4, DS7.4, DS8.4, HX711-1.1, HX711-1.7, HX711-2.1, HX711-3.1, HX711-4.1, HX711-4.7, HX711-5.1, I²C.4, LED.4, LM33CV_G2.2, LM33CV_G3.2, PCF8591_I²C.2, RASPBERRY_PI.9, SEEED1.4, SEEED2.4, SEEED3.4, SEEED4.4, SEEED5.4, TASTER_LED.4, UART_GROVE.4
- net 3V3: now also DS18_3V3/GPIO9.2; no longer JP_3V3_GPIO9.2
- net 3V3_PIN1: now also DS18_3V3/GPIO9.3; no longer JP_3V3_GPIO9.3
- net 3V3_PIN17: now also HX711_RPI/LM33.1; no longer JP_3V3_RPI/LM33_G3.1
- net 5V_1: now also 5V(ALTERN.IN).1, 5V(OUT).1; no longer 5V(ALTERN.).1
- net 5V_PIN2: now also C_HC711_1.1, LM33_HX711.1, LM33_I²C.1, RASPBERRY_PI.2; no longer C_SP5.1, LM33CV_G2.1, LM33CV_G3.1
- net DS18B20_3V3_GPIO9_PIN21: now also DS18_3V3/GPIO9.1; no longer JP_3V3_GPIO9.1
- net GND: now also #76_77.2, 32.-, 5V(ALTERN.IN).2, 5V(ALTERN.IN).3, 5V(OUT).2, 5V(OUT).3, BME680.2, BME680_GROVE.4, C1.-, C_HC711_1.2, C_I²C_1.2, C_TASTER.1, DS1.4, DS18B20(T0-92).1, DS18B20-1.3, DS18B20-2.3, DS18B20-3.3, DS18B20-4.3, DS18B20-5.3, DS18B20-6.3, DS18B20-7.3, DS18B20-8.3, DS2.4, DS3.4, DS4.4, DS5.4, DS6.4, DS7.4, DS8.4, HX711-1.1, HX711-1.7, HX711-2.1, HX711-3.1, HX711-4.1, HX711-4.7, HX711-5.1, I²C.4, LED.4, LM33_HX711.2, LM33_I²C.2, PCF8591_I²C.2, RASPBERRY_PI.9, SEEED1.4, SEEED2.4, SEEED3.4, SEEED4.4, SEEED5.4, TASTER_LED.4, UART_GROVE.4; no longer 5V(ALTERN.).3
- net HX711_V: now also HX.1, HX711_RPI/LM33.2; no longer JP_3V3_RPI/LM33_G3.2
- net N$2: now also C1.+, LM33_I²C.3; no longer C_SP4.1, LM33CV_G2.3
- net N$4: now also 32.+, HX711_RPI/LM33.3, LM33_HX711.3; no longer C_SP6.1, JP_3V3_RPI/LM33_G3.3, LM33CV_G3.3
- net N$8: now also #76_77.1; no longer 0#76/77.2
Routing:
- net GND_2: track 400.5 -> 0.00 mm
- net GND: track 72.6 -> 458.5 mm
- net 5V_PIN2: track 62.7 -> 106.2 mm, vias 0 -> 2
- net DS18B20_3V3_GPIO9_PIN21: track 53.5 -> 35.4 mm, vias 0 -> 1
- net N$10: track 17.9 -> 4.33 mm
- net 5V_1: track 71.3 -> 83.7 mm
- net DS18B20_DATA_GPIO11_PIN23: track 197.6 -> 186.3 mm
- net 3V3_PIN1: track 125.4 -> 136.6 mm, vias 2 -> 0
- net LED_2: track 23.9 -> 13.6 mm
- net BME_SCL/SCK_PIN5: track 155.9 -> 146.3 mm
- net LED_GPIO21_PIN40: track 24.5 -> 32.4 mm
- net HX711-SCK_GPIO24_PIN18: track 62.0 -> 69.0 mm
- net 3V3_PIN17: track 133.7 -> 127.3 mm
- net HX711_V: track 119.1 -> 125.4 mm
- net I²C_V: track 65.9 -> 70.6 mm
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Other:
- board text added: "3V3 (DT/DAT) (SCK) (GND)"
- board text added: "3V3 G2 G3 G4 GND G17 G27 G22 3v3 G10 G9 G11 GND IDSD G5 G6 G13 G19 G26 GND"
- board text added: "3V3 GND SCL SDA SDO"
- board text added: "5V 5V GND G14 G15 G18 GND G23 G24 GND G25 G8 G7 IDSC GND G12 GND G16 G20 G21"
- board text added: "GND DT SCK 3V3"
- board text added: "GND DT SCK 3V3 (DT/DAT) (SCK) (GND)"
- board text added: "HoneyPi HAT 2.01 https://www.honey-pi.de/"
- board text added: "SCL SDA GND 3.3V"
- board text added: "SDA SCL 3.3V GND"
- board text removed: "3.3V GND SDA SCL"
- board text removed: "GND SCK DT 3V3"
- board text removed: "GND SCK DT 3V3 (SCK) (DT) (GND)"
- board text removed: "HoneyPi HAT 2.0 https://www.honey-pi.de/"
- board text removed: "SCL SDA 3V3 GND SDO"
