File: PCB_V2.x/HoneyPI_Platine_2.01.brd (EAGLE design)
At the start: 80 x 100 mm, 81 parts

Commit message: 2x Polyfuse
The circuit has been extended by 2 optional polyfuses or similar.  The fuse size has been accepted and not yet verified.
Please note: The operator of the board must ensure safe operation. Accordingly, a fuse must be installed in accordance with the regulations.
Parts:
- added F1: 0,25A, fuse:TR5
- added F2: 0,5A, fuse:TR5
- added JP1: (no value), pinhead:1X07
- added JP2, JP3: (no value), pinhead:1X06
- moved C_SP1 13.5 mm to (21.6, 17.8)
- moved R_DS18B20 5.24 mm to (19.1, 38.1)
- moved C_SP2 2.84 mm to (21.6, 25.4)
- moved U$11 2.00 mm to (12.5, 52.0)
- moved DCIN- 0.76 mm to (20.3, 7.62)
- moved DC_OUT_5V- 0.76 mm to (20.3, 47.6)
- moved DCIN2- 0.32 mm to (22.9, 7.62)
- moved DC_OUT2_5V- 0.32 mm to (22.9, 57.6)
Connections:
- removed net N$45: DCIN+.1, POWER_IN.1, R1_PCF8591.1
- new net N$5: DCIN+.1, F1.1, R1_PCF8591.1
- new net N$7: F1.2, POWER_IN.1
- new net N$9: 5V(ALTERN.IN).1, F2.2
- net 5V_1: now also F2.1; no longer 5V(ALTERN.IN).1
Routing:
- net N$5: track 0.00 -> 72.9 mm
- net N$45: track 65.6 -> 0.00 mm
- net N$7: track 0.00 -> 22.9 mm
- net 3V3_PIN1: track 136.6 -> 113.8 mm
- net DS18B20_DATA_GPIO11_PIN23: track 186.3 -> 165.3 mm, vias 1 -> 2
- net BME_SCL/SCK_PIN5: track 146.3 -> 127.5 mm, vias 0 -> 2
- net BME_SDI/SDA_PIN3: track 150.4 -> 132.7 mm, vias 2 -> 1
- net N$9: track 0.00 -> 16.9 mm
- net 3V3_PIN17: track 127.3 -> 113.6 mm, vias 0 -> 1
- net 5V_1: track 83.7 -> 74.2 mm
- net HX711_V: track 125.4 -> 116.8 mm
- net HX711-SCK_GPIO24_PIN18: track 69.0 -> 60.7 mm
- net HX711-DT_GPIO5_PIN29: track 56.6 -> 51.1 mm, vias 0 -> 1
- net HX711-SCK_GPIO6_PIN31: track 61.6 -> 64.8 mm
- net GND: track 458.5 -> 461.6 mm, vias 1 -> 0
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