File: PCB_V2.x/HoneyPI_Platine_2.02.brd (EAGLE design)
At the start: 80 x 100 mm, 89 parts

Commit message: New releases
Fix BME680_GROVE Pinout on the main board
Some corrections on the sensor board
Parts:
- C_SP1: value 100µF -> xxµF
- C_SP2: value 1µF -> xµF
Connections:
- net BME_SCL/SCK_PIN5: now also BME680_GROVE.1; no longer BME680_GROVE.2
- net BME_SDI/SDA_PIN3: now also BME680_GROVE.2; no longer BME680_GROVE.1
Other:
- board text added: "(!) Pinout modified to 2.01! Check documentation."
- board text added: "GND 3.3V SDA(!) SCL(!)"
- board text added: "HoneyPi HAT 2.02 https://www.honey-pi.de"
- board text added: "LED- NotC NotC LED+"
- board text removed: "GND 3.3V SDA SCL"
- board text removed: "GND 3v3"
- board text removed: "HoneyPi HAT 2.01 https://www.honey-pi.de"
Changed lines of the file:
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@@
 </layers>
 <board>
-<fusionsync huburn="a.cGVyc29uYWw6dWUyYjlkYjlm" projecturn="a.cGVyc29uYWw6dWUyYjlkYjlmIzIwMTcwNDEzNzE3MzExMDE" f3durn="urn:adsk.wipprod:dm.lineage:GkcBSzvJT7K4Bick1Iit8w" pcbguid="" lastpulledtime="" lastsyncedchangeguid="" latestrevisionid="f7b36f48-5fd6-4382-b252-79246711c0d3" lastsyncedrevisionid="f7b36f48-5fd6-4382-b252-79246711c0d3" lastboardhashguid="1bca5865-5669-4ab1-a0ca-56b80251d355" lastpushedtime="2020-06-08T22:28:48Z" linktopcb3d="true"/>
+<fusionsync huburn="a.cGVyc29uYWw6dWUyYjlkYjlm" projecturn="a.cGVyc29uYWw6dWUyYjlkYjlmIzIwMTcwNDEzNzE3MzExMDE" f3durn="urn:adsk.wipprod:dm.lineage:GkcBSzvJT7K4Bick1Iit8w" pcbguid="" lastpulledtime="" lastsyncedchangeguid="" latestrevisionid="f7b36f48-5fd6-4382-b252-79246711c0d3" lastsyncedrevisionid="f7b36f48-5fd6-4382-b252-79246711c0d3" lastboardhashguid="1bca5865-5669-4ab1-a0ca-56b80251d355" lastpushedtime="2020-06-08T22:28:48Z" linktopcb3d="false"/>
 <plain>
 <wire x1="0" y1="0" x2="80" y2="0" width="0" layer="20"/>
@@
 <wire x1="0" y1="100" x2="0" y2="0" width="0" layer="20"/>
 <hole x="2.54" y="94.234" drill="3" locked="yes" grouprefs="RASPBERRY"/>
-<hole x="2.54" y="71.374" drill="3" grouprefs="RASPBERRY HX711_1"/>
+<hole x="2.54" y="71.374" drill="3" grouprefs="HX711_1 RASPBERRY"/>
 <text x="13.843" y="77.216" size="0.8128" layer="25" rot="R180" grouprefs="HX711_1">3V3
 (DT/DAT)
@@
 3V3
 DATA</text>
-<text x="54.71" y="7.374" size="1.27" layer="1" font="vector" ratio="12">HoneyPi HAT 2.01
+<text x="54.71" y="7.374" size="1.27" layer="25" font="vector" ratio="12">HoneyPi HAT 2.02
 https://www.honey-pi.de </text>
 <text x="78.543" y="87.992" size="0.8128" layer="25" rot="R90" grouprefs="HX711_4">GND
@@
 DT
 SCK</text>
-<text x="51.308" y="69.596" size="0.6604" layer="25" rot="R90">GND
-3v3</text>
+<text x="51.308" y="69.596" size="0.6604" layer="25" rot="R90">LED-
+ NotC
+ NotC
+LED+</text>
 <text x="37.973" y="64.77" size="0.762" layer="25">PIN3
  |  LM 3v3
@@
 GND</text>
 <hole x="77.47" y="20.54" drill="3"/>
-<text x="66.167" y="21.082" size="0.8128" layer="25" rot="R90">GND
+<text x="66.167" y="20.682" size="0.8128" layer="25" rot="R90">GND
 3.3V
-SDA
-SCL
+SDA(!)
+SCL(!)
 </text>
 <hole x="2.54" y="52" drill="3"/>
@@
 <text x="6.096" y="11.684" size="1.7018" layer="25" rot="R180">-</text>
 <text x="6.096" y="21.082" size="1.7018" layer="25">-</text>
+<text x="56.41" y="3.474" size="0.8128" layer="25" font="vector" ratio="12">(!) Pinout modified to 2.01!
+Check documentation.</text>
 </plain>
 <attributes>
@@
 <attribute name="VALUE" x="43.18" y="59.563" size="1.27" layer="27"/>
 </element>
-<element name="C_SP1" library="capacitor-wima" library_urn="urn:adsk.eagle:library:116" package="C2.5-3" package3d_urn="urn:adsk.eagle:package:5436/1" value="100µF" x="21.59" y="17.78" smashed="yes" rot="R270">
+<element name="C_SP1" library="capacitor-wima" library_urn="urn:adsk.eagle:library:116" package="C2.5-3" package3d_urn="urn:adsk.eagle:package:5436/1" value="xxµF" x="21.59" y="17.78" smashed="yes" rot="R270">
 <attribute name="NAME" x="23.368" y="19.431" size="0.8128" layer="25" ratio="10" rot="R270"/>
 <attribute name="POPULARITY" value="38" x="21.59" y="16.51" size="0.8128" layer="27" rot="R270" display="off"/>
 <attribute name="VALUE" x="18.542" y="19.431" size="0.8128" layer="27" ratio="10" rot="R270"/>
 </element>
-<element name="C_SP2" library="capacitor-wima" library_urn="urn:adsk.eagle:library:116" package="C2.5-3" package3d_urn="urn:adsk.eagle:package:5436/1" value="1µF" x="21.59" y="25.4" smashed="yes" rot="R270">
+<element name="C_SP2" library="capacitor-wima" library_urn="urn:adsk.eagle:library:116" package="C2.5-3" package3d_urn="urn:adsk.eagle:package:5436/1" value="xµF" x="21.59" y="25.4" smashed="yes" rot="R270">
 <attribute name="NAME" x="23.368" y="27.051" size="0.8128" layer="25" ratio="10" rot="R270"/>
 <attribute name="POPULARITY" value="38" x="21.59" y="26.67" size="0.8128" layer="27" rot="R270" display="off"/>
@@
 <contactref element="I²C" pad="2"/>
 <contactref element="BME680" pad="3"/>
-<contactref element="BME680_GROVE" pad="2"/>
 <contactref element="PCF8591_I²C" pad="4"/>
 <wire x1="62.1792" y1="26.7208" x2="61.976" y2="26.7208" width="0.1524" layer="16"/>
@@
 <wire x1="70.5104" y1="28.5496" x2="64.008" y2="28.5496" width="0.1524" layer="16"/>
 <wire x1="72.39" y1="26.67" x2="70.5104" y2="28.5496" width="0.1524" layer="16"/>
-<wire x1="61.976" y1="26.7208" x2="61.96" y2="26.67" width="0.1524" layer="16"/>
 <wire x1="5.8928" y1="85.852" x2="12.7" y2="92.6592" width="0.1524" layer="16"/>
 <wire x1="5.7912" y1="85.852" x2="5.8928" y2="85.852" width="0.1524" layer="16"/>
@@
 <wire x1="50.0888" y1="24.7904" x2="59.5376" y2="24.7904" width="0.1524" layer="16"/>
 <wire x1="48.26" y1="26.6192" x2="50.0888" y2="24.7904" width="0.1524" layer="16"/>
-<wire x1="61.8744" y1="26.6192" x2="61.96" y2="26.67" width="0.1524" layer="16"/>
 <wire x1="48.26" y1="26.6192" x2="48.26" y2="26.67" width="0.1524" layer="16"/>
+<contactref element="BME680_GROVE" pad="1"/>
+<wire x1="61.976" y1="26.7208" x2="63.96" y2="26.67" width="0" layer="19" extent="16-16"/>
+<wire x1="61.8744" y1="26.6192" x2="61.976" y2="26.7208" width="0" layer="19" extent="16-16"/>
 </signal>
 <signal name="HX711_V" class="1">
@@
 <contactref element="BME680" pad="4"/>
 <contactref element="PCF8591_I²C" pad="3"/>
-<contactref element="BME680_GROVE" pad="1"/>
 <wire x1="69.7992" y1="26.7208" x2="64.008" y2="26.7208" width="0.1524" layer="1"/>
-<wire x1="64.008" y1="26.7208" x2="63.96" y2="26.67" width="0.1524" layer="1"/>
 <wire x1="69.7992" y1="26.7208" x2="69.85" y2="26.67" width="0.1524" layer="1"/>
 <wire x1="51.0032" y1="26.6192" x2="50.8" y2="26.6192" width="0.1524" layer="1"/>
@@
 <wire x1="63.9064" y1="26.6192" x2="62.0776" y2="24.7904" width="0.1524" layer="1"/>
 <wire x1="50.8" y1="26.6192" x2="50.8" y2="26.67" width="0.1524" layer="1"/>
-<wire x1="63.9064" y1="26.6192" x2="63.96" y2="26.67" width="0.1524" layer="1"/>
 <wire x1="10.16" y1="90.8304" x2="10.16" y2="92.71" width="0.1524" layer="16"/>
 <wire x1="4.2672" y1="84.9376" x2="10.16" y2="90.8304" width="0.1524" layer="16"/>
@@
 <wire x1="52.7304" y1="24.7904" x2="52.7812" y2="24.8412" width="0.1524" layer="1"/>
 <wire x1="40.64" y1="14.6304" x2="40.64" y2="14.605" width="0.1524" layer="1"/>
+<contactref element="BME680_GROVE" pad="2"/>
+<wire x1="63.9064" y1="26.6192" x2="64.008" y2="26.7208" width="0" layer="19" extent="1-1"/>
+<wire x1="61.96" y1="26.67" x2="63.9064" y2="26.6192" width="0" layer="19" extent="1-1"/>
 </signal>
 <signal name="N$2">
