File: PCB_TimerBoard_2.x/HoneyPI_Platine TimerBoard 2.00a.sch (EAGLE design)
At the start: 23 parts, among them Q1 NDP6020P, Q2 BC547, Q3 BC547, Q4 NDP6020P, Q5 BC547, Q6 BC547

Commit message: RC
Parts:
- removed C1: 0,1µF, capacitor-wima:C2,5-3
- removed C4: 10µF, rcl:CPOL-EUE2-5
- removed DS2, ZS-042(DS3231): (no value), pinhead:PINHD-1X5
- removed LM33CV: (no value), LM33cv:LM337TS
- removed NO_CONECTION: (no value), pinhead:PINHD-1X4
- removed Q1: NDP6020P, transistor-power:IRF9530
- removed Q2, Q3: BC547, transistor-npn:BC338
- removed R1, R2: 10k, rcl:R-EU_0204/7
- removed RPI_ON1: (no value), special:SW_DIP-1
- added JP3: (no value), pinhead:PINHD-1X1
Connections:
- removed net ALARM_SQW_2: Q2.B, RPI_ON1.2, ZS-042(DS3231).1
- removed net GND_2: C1.1, C4.-, DS2.3, LM33CV.IN, Q2.E, Q3.E, RPI_ON1.1, ZS-042(DS3231).5
- removed net N$5: Q1.G, Q3.C, R1.1
- removed net N$6: Q2.C, Q3.B, R2.2
- removed net SCL/SCK_PIN5_2: DS2.5, ZS-042(DS3231).2
- removed net SDI/SDA_PIN3_2: DS2.4, ZS-042(DS3231).3
- removed net V_IN_5V_2: C1.2, DS2.1, LM33CV.GND, Q1.S, R1.2, R2.1
- removed net V_LF33CV: C4.+, LM33CV.OUT3V3, ZS-042(DS3231).4
- removed net V_OUT_5V_2: DS2.2, Q1.D
Other:
- moved on the sheet: A_5V, B_3V3, DS1, NO_CONECTION1, Q4, Q5, Q6, R3, R4, RPI_ON2, ZS-042(DS3231)1
