File: PCB_V2.x/OLD/HoneyPI_Platine_2.01.brd (EAGLE design)
At the start: 80 x 100 mm, 89 parts

Commit message: Release
Parts:
- removed HX1, HX2, HX3: (no value), pinhead:1X01
- removed JP_R_LED: (no value), pinhead:1X02
- removed U$13: (no value), holes:3,0
- added DS18_3V3/GPIO9, JP_VORW: (no value), pinhead:1X03
- R_LED: value 130Ohm -> 130
- moved UART_GROVE 3.05 mm to (68.3, 97.2), turned to 0 degrees
- moved HX711-4 1.20 mm to (69.8, 86.4)
- renumbered C_HX711_1 to C_HC711_1, C_HX711_2 to 32, C_I²C_2 to C1, GROVE1 to SEEED1, GROVE2 to SEEED2, GROVE3 to SEEED3, GROVE4 to SEEED4, GROVE5 to SEEED5, LF33_HX711 to LM33_HX711, LF33_I²C to LM33_I²C
Connections:
- net GND20V renamed N$1
- net SPANNUNGSTEILER1 renamed N$6
- net VDD20V1 renamed N$5
- net VDD20V2 renamed N$7
- new net N$10: JP_VORW.1, R_LED.1
- net 3V3: now also DS18_3V3/GPIO9.2; no longer HX2.1
- net 3V3_PIN1: now also DS18_3V3/GPIO9.3; no longer HX3.1
- net DS18B20_3V3_GPIO9_PIN21: now also DS18_3V3/GPIO9.1; no longer HX1.1
- net LED_2: now also JP_VORW.3; no longer JP_R_LED.2
- net LED_GPIO21_PIN40: now also JP_VORW.2; no longer JP_R_LED.1, R_LED.1
Routing:
- net DS18B20_3V3_GPIO9_PIN21: track 58.0 -> 36.1 mm, vias 0 -> 1
- net 3V3_PIN17: track 93.9 -> 113.6 mm
- net BME_SCL/SCK_PIN5: track 140.9 -> 127.5 mm, vias 0 -> 2
- net 3V3_PIN1: track 125.3 -> 113.8 mm, vias 1 -> 0
- net HX711-DT_GPIO5_PIN29: track 59.6 -> 51.1 mm, vias 0 -> 1
- net HX711-DT_GPIO23_PIN16: track 69.2 -> 61.1 mm
- net LED_GPIO21_PIN40: track 39.3 -> 32.4 mm
- net BME_SDI/SDA_PIN3: track 139.3 -> 132.7 mm, vias 0 -> 1
- net RX_0_PIN_10: track 54.8 -> 48.9 mm
- net HX711_V: track 122.5 -> 116.8 mm, vias 1 -> 2
- net DS18B20_DATA_GPIO11_PIN23: track 160.7 -> 165.3 mm
- net N$10: track 0.00 -> 4.33 mm
- net 3V3: track 138.5 -> 134.5 mm
- net I²C_V: track 67.0 -> 70.9 mm
- net TX_0_PIN_8: track 57.5 -> 53.8 mm
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