File: PCB_V2.x/OLD/HoneyPI_Platine_2.01.sch (EAGLE design)
At the start: 76 parts

Commit message: Release
Parts:
- removed C_HX711_1: 0,1µF, capacitor-wima:C2,5-3
- removed C_HX711_2: 10µF, rcl:CPOL-EUE2-5
- removed HX1, HX2, HX3: (no value), pinhead:PINHD-1X1
- removed JP_R_LED: (no value), pinhead:PINHD-1X2
- removed LF33_HX711: (no value), LM33cv:LM33CV
- added 32: 10µF, rcl:CPOL-EUE2-5
- added C_HC711_1: 0,1µF, capacitor-wima:C2,5-3
- added DS18_3V3/GPIO9, JP_VORW: (no value), pinhead:PINHD-1X3
- added LM33_HX711: (no value), LM33cv:LM33CV
- R_LED: value 130Ohm -> 130; POPULARITY 130Ohm -> 130
- renumbered C_I²C_2 to C1, GROVE1 to SEEED1, GROVE2 to SEEED2, GROVE3 to SEEED3, GROVE4 to SEEED4, GROVE5 to SEEED5, LF33_I²C to LM33_I²C
Connections:
- net GND20V renamed N$1
- net SPANNUNGSTEILER1 renamed N$6
- net VDD20V1 renamed N$5
- net VDD20V2 renamed N$7
- new net N$10: JP_VORW.1, R_LED.1
- net 3V3: now also DS18_3V3/GPIO9.2; no longer HX2.1
- net 3V3_PIN1: now also DS18_3V3/GPIO9.3; no longer HX3.1
- net 5V_PIN2: now also C_HC711_1.1, LM33_HX711.5V; no longer C_HX711_1.1, LF33_HX711.5V
- net DS18B20_3V3_GPIO9_PIN21: now also DS18_3V3/GPIO9.1; no longer HX1.1
- net GND: now also 32.-, C_HC711_1.2, LM33_HX711.GND; no longer C_HX711_1.2, C_HX711_2.-, LF33_HX711.GND
- net LED_2: now also JP_VORW.3; no longer JP_R_LED.2
- net LED_GPIO21_PIN40: now also JP_VORW.2; no longer JP_R_LED.1, R_LED.1
- net N$4: now also 32.+, LM33_HX711.OUT3V3; no longer C_HX711_2.+, LF33_HX711.OUT3V3
Other:
- note added: "Die Spannungsversorgung 3v3 kann vom Raspberry Pi oder von einem Festspannungsregler, wie z.B. dem LM33CV, kommen. Der LM33CV bekommt 5V vom Spannungsversorgungsteil. JP: 1-2 Raspberry Pi (Pin17) JP: 2-3 LM33CV"
- note added: "GPIO09"
- note added: "HX711 Es gibt verschiedene HX711 Module. Damit diese angeschlossen werden können, wurden 3 verschiedene Belegungen realisiert und mit Grün, Pflaume und SEEED gekennzeichnet. Grün: Für das grüne Modul ( u.a. über Aliexpress, Ebay) Plaume: für das pflaumenfarbige Modul (u.a. Aliexpress, Ebay) Seeed: Modul mit Grove vorgefertigt https://www.seeedstudio.com Auf der Platine werden die Löcher so eng ge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"
- note removed: "Die Spannungsversorgung 3v3 kann vom Raspberry Pi oder von einem Festspannungsregler, wie z.B. dem Lf33CV, kommen. Der Lf33CV bekommt 5V vom Spannungsversorgungsteil. JP: 1-2 Raspberry Pi (Pin17) JP: 2-3 Lf33CV"
- note removed: "HX711 Es gibt verschiedene HX711 Module. Damit diese angeschlossen werden können, wurden 3 verschiedene Belegungen realisiert und mit Grün, Pflaume und Grove gekennzeichnet. Grün: Für das grüne Modul ( u.a. über Aliexpress, Ebay) Plaume: für das pflaumenfarbige Modul (u.a. Aliexpress, Ebay) Grove: Steckverbinder für Modul mit Grove (vorgefertigt) https://www.seeedstudio.com Auf der Platine werden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"
- moved on the sheet: #76_77, BME680, BME680_GROVE, C_TASTER, HX, HX711_RPI/LM33, I²C, LED, PCF8591_I²C, R_LED, R_TASTER, S_TASTER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
