File: PCB_Sensor_Board_2.x_BME280_680_ATH10_HDC1080/PCB_Sensor_Board_2.x_BME280_680_ATH10_HDC1080.brd (EAGLE design)
At the start: 30 x 62 mm, 10 parts

Commit message: Gerber update
Parts:
- removed GND, JP1_ANSCHLUSS, OTHER, OTHER1: (no value), pinhead:1X04
- added HDC1080, SHT31/ATH10: (no value), pinhead:1X04
- added X1: (no value), con-wago:233-504
- moved J1 1.80 mm to (11.4, 52.1)
Connections:
- net 3V3: now also HDC1080.2, SHT31/ATH10.1, X1.B1; no longer JP1_ANSCHLUSS.1, OTHER.4, OTHER1.4
- net BME_SCL/SCK: now also HDC1080.4, SHT31/ATH10.3, X1.B3; no longer JP1_ANSCHLUSS.3, OTHER.2, OTHER1.2
- net BME_SDI/SDA: now also HDC1080.3, SHT31/ATH10.4, X1.B4; no longer JP1_ANSCHLUSS.4, OTHER.1, OTHER1.1
- net GND: now also HDC1080.1, SHT31/ATH10.2, X1.B2; no longer GND.1, GND.2, GND.3, GND.4, JP1_ANSCHLUSS.2, OTHER.3, OTHER1.3
Routing:
- net GND: track 70.1 -> 54.2 mm
- net 3V3: track 59.2 -> 52.7 mm
- net BME_SCL/SCK: track 54.2 -> 56.0 mm

Commit message: Update
Parts:
- removed BME680/280, SHT31/ATH10: (no value), pinhead:1X04
- added BME680, SHT31/ATH10/BME280: (no value), pinhead:1X04
- moved HDC1080 43.1 mm to (20.3, 53.3), turned to 90 degrees
- moved J1 41.9 mm to (12.7, 10.2), turned to 270 degrees
- moved X1 41.9 mm to (19.1, 10.2), turned to 90 degrees
Connections:
- net 3V3: now also BME680.1, SHT31/ATH10/BME280.1; no longer BME680/280.1, SHT31/ATH10.1
- net BME_SCL/SCK: now also BME680.3, SHT31/ATH10/BME280.3; no longer BME680/280.3, SHT31/ATH10.3
- net BME_SDI/SDA: now also BME680.4, SHT31/ATH10/BME280.4; no longer BME680/280.4, SHT31/ATH10.4
- net GND: now also BME680.2, SHT31/ATH10/BME280.2; no longer BME680/280.2, SHT31/ATH10.2
Routing:
- net 3V3: track 52.7 -> 83.0 mm
- net BME_SCL/SCK: track 56.0 -> 61.5 mm
- net GND: track 54.2 -> 58.6 mm
- net BME_SDI/SDA: track 52.3 -> 56.5 mm
Other:
- board text added: "3v3"
- board text added: "BME680/280 Sensor Board 2.01 https://www.honey-pi.de/"
- board text added: "GND"
- board text added: "SCL SDA"
- board text added: "SCL SDA 3v3 GND"
- board text added: "SDA SCL GND 3v3"
- board text removed: "HoneyPI_Platine_2.0_BME680_280_Sensor_Board https://www.honey-pi.de/"

Commit message: Update
Routing:
- net 3V3: track 83.0 -> 65.4 mm
- net GND: track 58.6 -> 61.7 mm
