File: PCB_Sensor_Board_2.x_BME280_680_ATH10_HDC1080/PCB_Sensor_Board_2.x_BME280_680_ATH10_HDC1080.sch (EAGLE design)
At the start: 6 parts

Commit message: Gerber update
Parts:
- removed GND, JP1_ANSCHLUSS, OTHER, OTHER1: (no value), pinhead:PINHD-1X4
- added HDC1080, SHT31/ATH10: (no value), pinhead:PINHD-1X4
- added X1: (no value), con-wago:233-504
Connections:
- net 3V3: now also HDC1080.2, SHT31/ATH10.1, X1.B-1; no longer JP1_ANSCHLUSS.1, OTHER.4, OTHER1.4
- net BME_SCL/SCK: now also HDC1080.4, SHT31/ATH10.3, X1.B-3; no longer JP1_ANSCHLUSS.3, OTHER.2, OTHER1.2
- net BME_SDI/SDA: now also HDC1080.3, SHT31/ATH10.4, X1.B-4; no longer JP1_ANSCHLUSS.4, OTHER.1, OTHER1.1
- net GND: now also HDC1080.1, SHT31/ATH10.2, X1.B-2; no longer GND.1, GND.2, GND.3, GND.4, JP1_ANSCHLUSS.2, OTHER.3, OTHER1.3
Other:
- moved on the sheet: BME680/280

Commit message: Update
Parts:
- removed BME680/280, SHT31/ATH10: (no value), pinhead:PINHD-1X4
- added BME680, SHT31/ATH10/BME280: (no value), pinhead:PINHD-1X4
Connections:
- net 3V3: now also BME680.1, SHT31/ATH10/BME280.1; no longer BME680/280.1, SHT31/ATH10.1
- net BME_SCL/SCK: now also BME680.3, SHT31/ATH10/BME280.3; no longer BME680/280.3, SHT31/ATH10.3
- net BME_SDI/SDA: now also BME680.4, SHT31/ATH10/BME280.4; no longer BME680/280.4, SHT31/ATH10.4
- net GND: now also BME680.2, SHT31/ATH10/BME280.2; no longer BME680/280.2, SHT31/ATH10.2
Other:
- moved on the sheet: HDC1080
